File: supply/shinobi_5v_3V3.brd (EAGLE design)
At the start: 40.5 x 35 mm, 7 parts

Commit message: Update Shinobi.
Other:
- board text added: "Rev 1.0.0.A"
- board text removed: "Rev 1.0.0.Beta2"
Changed lines of the file:
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@@
 <?xml version="1.0" encoding="utf-8"?>
 <!DOCTYPE eagle SYSTEM "eagle.dtd">
-<eagle version="8.2.2">
+<eagle version="8.5.1">
 <drawing>
 <settings>
 <setting alwaysvectorfont="no"/>
+<setting keepoldvectorfont="yes"/>
 <setting verticaltext="up"/>
 </settings>
@@
 <text x="5.892" y="27.186" size="1.27" layer="21">USB Battery(5V-&gt;3V3)</text>
 <text x="12.692" y="29.286" size="2.54" layer="21">#8</text>
-<text x="5.892" y="25.786" size="0.6096" layer="21">Rev 1.0.0.Beta2</text>
+<text x="5.892" y="25.786" size="0.6096" layer="21">Rev 1.0.0.A</text>
 </plain>
 <attributes>
@@
 <param name="dpMaxLengthDifference" value="10mm"/>
 <param name="dpGapFactor" value="2.5"/>
-<param name="checkGrid" value="0"/>
 <param name="checkAngle" value="0"/>
 <param name="checkFont" value="1"/>
 <param name="checkRestrict" value="1"/>
+<param name="checkStop" value="0"/>
+<param name="checkValues" value="0"/>
 <param name="useDiameter" value="13"/>
 <param name="maxErrors" value="50"/>
