File: supply/shinobi_5v_3V3_dcdc_jack.brd (EAGLE design)
At the start: 40.5 x 35 mm, 13 parts, among them IC1 LM3671, P1 POLYSWITCH1210

Commit message: Update Shinobi.
Parts:
- moved P4 2.60 mm to (36.0, 18.2)
- moved P1 2.40 mm to (27.1, 21.6)
- moved M1 2.11 mm to (22.2, 21.8)
- moved R1 1.22 mm to (17.9, 18.2), turned to 90 degrees
- moved C10 0.90 mm to (24.7, 14.5)
- moved L1 0.82 mm to (14.7, 17.9)
- moved C2 0.80 mm to (12.5, 18.1)
- moved C3 0.80 mm to (24.7, 12.0)
Routing:
- net 5V: track 25.8 -> 23.0 mm
- net N$1: track 4.31 -> 5.43 mm
- net N$2: track 5.93 -> 6.63 mm
- net N$15: track 7.14 -> 7.70 mm
Other:
- board text added: "Rev 1.0.0.B"
- board text removed: "Rev 1.0.0.A"
Changed lines of the file:
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@@
 <?xml version="1.0" encoding="utf-8"?>
 <!DOCTYPE eagle SYSTEM "eagle.dtd">
-<eagle version="8.2.2">
+<eagle version="8.5.1">
 <drawing>
 <settings>
 <setting alwaysvectorfont="no"/>
+<setting keepoldvectorfont="yes"/>
 <setting verticaltext="up"/>
 </settings>
-<grid distance="0.1" unitdist="mm" unit="mm" style="lines" multiple="1" display="no" altdistance="5" altunitdist="mil" altunit="mil"/>
+<grid distance="0.01" unitdist="mm" unit="mm" style="lines" multiple="1" display="no" altdistance="5" altunitdist="mil" altunit="mil"/>
 <layers>
 <layer number="1" name="Top" color="4" fill="1" visible="yes" active="yes"/>
@@
 <text x="5.892" y="27.186" size="1.27" layer="21">DC Battery(5V-&gt;3V3 DCDC)</text>
 <text x="12.692" y="29.286" size="2.54" layer="21">#9</text>
-<text x="5.892" y="25.786" size="0.6096" layer="21">Rev 1.0.0.A</text>
+<text x="5.892" y="25.786" size="0.6096" layer="21">Rev 1.0.0.B</text>
 </plain>
 <attributes>
@@
 <param name="dpMaxLengthDifference" value="10mm"/>
 <param name="dpGapFactor" value="2.5"/>
-<param name="checkGrid" value="0"/>
 <param name="checkAngle" value="0"/>
 <param name="checkFont" value="1"/>
 <param name="checkRestrict" value="1"/>
+<param name="checkStop" value="0"/>
+<param name="checkValues" value="0"/>
 <param name="useDiameter" value="13"/>
 <param name="maxErrors" value="50"/>
@@
 <element name="U$3" library="FaBo-Template" package="FABO-SHINOBI" value="" x="0" y="0"/>
 <element name="C1" library="FaBo-Capacitor" package="0603" value="4.7uF" x="21.9" y="13.6" rot="R270"/>
-<element name="C2" library="FaBo-Capacitor" package="0603" value="10uF" x="13.3" y="18.1" rot="R90"/>
+<element name="C2" library="FaBo-Capacitor" package="0603" value="10uF" x="12.5" y="18.1" rot="R90"/>
 <element name="IC1" library="FaBo-Supply" package="LM3671" value="LM3671" x="17.9" y="13.9" rot="R180"/>
-<element name="L1" library="FaBo-Coil" package="2.4X2.4" value="2.2uH" x="15.5" y="18.1"/>
-<element name="C10" library="FaBo-Capacitor" package="0603" value="0.1uF" x="25.6" y="14.5"/>
-<element name="C3" library="FaBo-Capacitor" package="0603" value="10uF" x="25.5" y="12"/>
-<element name="R1" library="FaBo-Resistors" package="0603" value="100K" x="18.9" y="18.9"/>
-<element name="M1" library="FaBo-Transistor" package="AOD417" value="" x="24.3" y="22"/>
-<element name="P4" library="FaBo-Supply" package="2DC-G213-B66" value="" x="38.6" y="18.2" rot="R270"/>
-<element name="P1" library="FaBo-Supply" package="1210" value="POLYSWITCH1210" x="29.5" y="21.7" rot="R90"/>
+<element name="L1" library="FaBo-Coil" package="2.4X2.4" value="2.2uH" x="14.7" y="17.9"/>
+<element name="C10" library="FaBo-Capacitor" package="0603" value="0.1uF" x="24.7" y="14.5"/>
+<element name="C3" library="FaBo-Capacitor" package="0603" value="10uF" x="24.7" y="12"/>
+<element name="R1" library="FaBo-Resistors" package="0603" value="100K" x="17.9" y="18.2" rot="R90"/>
+<element name="M1" library="FaBo-Transistor" package="AOD417" value="" x="22.2" y="21.8"/>
+<element name="P4" library="FaBo-Supply" package="2DC-G213-B66" value="" x="36" y="18.2" rot="R270"/>
+<element name="P1" library="FaBo-Supply" package="1210" value="POLYSWITCH1210" x="27.1" y="21.6" rot="R90"/>
 </elements>
 <signals>
@@
 <contactref element="R1" pad="1"/>
 <contactref element="M1" pad="S"/>
-<wire x1="26.586" y1="17.9" x2="26.586" y2="14.636" width="0.8128" layer="1"/>
-<wire x1="26.586" y1="14.636" x2="26.45" y2="14.5" width="0.8128" layer="1"/>
-<wire x1="26.45" y1="14.5" x2="26.45" y2="12.1" width="0.8128" layer="1"/>
-<wire x1="26.45" y1="12.1" x2="26.35" y2="12" width="0.8128" layer="1"/>
-<wire x1="26.35" y1="12" x2="26.35" y2="9.55" width="0.8128" layer="1"/>
-<wire x1="26.35" y1="9.55" x2="26.5" y2="9.4" width="0.8128" layer="1"/>
-<wire x1="26.5" y1="9.4" x2="23" y2="9.4" width="0.8128" layer="1"/>
+<wire x1="24.486" y1="17.7" x2="25.586" y2="14.536" width="0.8128" layer="1"/>
+<wire x1="25.586" y1="14.536" x2="25.55" y2="14.5" width="0.8128" layer="1"/>
+<wire x1="25.55" y1="14.5" x2="25.55" y2="12" width="0.8128" layer="1"/>
+<wire x1="25.55" y1="12" x2="25.55" y2="9.35" width="0.8128" layer="1"/>
+<wire x1="25.55" y1="9.35" x2="25.4" y2="9.4" width="0.8128" layer="1"/>
+<wire x1="25.4" y1="9.4" x2="23" y2="9.4" width="0.8128" layer="1"/>
 <wire x1="23" y1="9.4" x2="21.9" y2="10.5" width="0.8128" layer="1"/>
 <wire x1="21.9" y1="10.5" x2="21.9" y2="12.75" width="0.8128" layer="1"/>
 <wire x1="21.9" y1="12.75" x2="19.45" y2="12.75" width="0.6096" layer="1"/>
 <wire x1="19.45" y1="12.75" x2="19.25" y2="12.95" width="0.6096" layer="1"/>
-<wire x1="18.1356" y1="14.478" x2="18.1356" y2="18.8976" width="0.1524" layer="1"/>
-<wire x1="17.9832" y1="14.3256" x2="18.1356" y2="14.478" width="0.1524" layer="1"/>
-<wire x1="17.9832" y1="13.4112" x2="17.9832" y2="14.3256" width="0.1524" layer="1"/>
+<wire x1="17.9356" y1="14.478" x2="17.9356" y2="16.7976" width="0.1524" layer="1"/>
+<wire x1="17.9532" y1="13.7256" x2="17.9356" y2="14.478" width="0.1524" layer="1"/>
+<wire x1="17.9832" y1="13.4112" x2="17.9532" y2="13.7256" width="0.1524" layer="1"/>
 <wire x1="18.4404" y1="12.954" x2="17.9832" y2="13.4112" width="0.1524" layer="1"/>
 <wire x1="19.05" y1="12.954" x2="18.4404" y2="12.954" width="0.1524" layer="1"/>
-<wire x1="18.1356" y1="18.8976" x2="18.05" y2="18.9" width="0.1524" layer="1"/>
+<wire x1="17.9356" y1="16.7976" x2="17.9" y2="17.35" width="0.1524" layer="1"/>
 <wire x1="19.05" y1="12.954" x2="19.25" y2="12.95" width="0.1524" layer="1"/>
 </signal>
@@
 <contactref element="C2" pad="2"/>
 <wire x1="16.55" y1="14.85" x2="16.55" y2="17.775" width="0.6096" layer="1"/>
-<wire x1="16.55" y1="17.775" x2="16.225" y2="18.1" width="0.6096" layer="1"/>
-<wire x1="16.225" y1="18.1" x2="16.225" y2="20.575" width="0.6096" layer="1"/>
-<wire x1="16.225" y1="20.575" x2="16.1" y2="20.7" width="0.6096" layer="1"/>
-<wire x1="16.1" y1="20.7" x2="15.05" y2="20.7" width="0.6096" layer="1"/>
-<wire x1="15.05" y1="20.7" x2="13.3" y2="18.95" width="0.6096" layer="1"/>
-<wire x1="13.3" y1="18.95" x2="6.7716" y2="18.95" width="0.6096" layer="1"/>
+<wire x1="16.55" y1="17.775" x2="15.425" y2="17.9" width="0.6096" layer="1"/>
+<wire x1="15.425" y1="17.9" x2="15.525" y2="20.575" width="0.6096" layer="1"/>
+<wire x1="15.525" y1="20.575" x2="15.4" y2="20.7" width="0.6096" layer="1"/>
+<wire x1="15.4" y1="20.7" x2="14.05" y2="20.7" width="0.6096" layer="1"/>
+<wire x1="14.05" y1="20.7" x2="12.5" y2="18.95" width="0.6096" layer="1"/>
+<wire x1="12.5" y1="18.95" x2="6.7716" y2="18.95" width="0.6096" layer="1"/>
 <wire x1="6.7716" y1="18.95" x2="6.7216" y2="19" width="0.6096" layer="1"/>
 </signal>
@@
 <wire x1="14.7828" y1="17.9832" x2="14.7828" y2="15.0876" width="0.1524" layer="1"/>
 <wire x1="16.4592" y1="12.954" x2="16.55" y2="12.95" width="0.1524" layer="1"/>
-<wire x1="14.7828" y1="17.9832" x2="14.775" y2="18.1" width="0.1524" layer="1"/>
+<wire x1="14.7828" y1="17.9832" x2="13.975" y2="17.9" width="0.1524" layer="1"/>
 </signal>
 <signal name="N$1">
 <contactref element="IC1" pad="3"/>
 <contactref element="R1" pad="2"/>
-<wire x1="19.3548" y1="17.8308" x2="19.3548" y2="14.9352" width="0.1524" layer="1"/>
-<wire x1="19.6596" y1="18.1356" x2="19.3548" y2="17.8308" width="0.1524" layer="1"/>
-<wire x1="19.6596" y1="18.8976" x2="19.6596" y2="18.1356" width="0.1524" layer="1"/>
-<wire x1="19.3548" y1="14.9352" x2="19.25" y2="14.85" width="0.1524" layer="1"/>
-<wire x1="19.6596" y1="18.8976" x2="19.75" y2="18.9" width="0.1524" layer="1"/>
+<wire x1="18.7548" y1="17.0308" x2="18.7548" y2="14.9252" width="0.1524" layer="1"/>
+<wire x1="18.7596" y1="18.9956" x2="18.7548" y2="17.0308" width="0.1524" layer="1"/>
+<wire x1="18.5596" y1="18.9976" x2="18.7596" y2="18.9956" width="0.1524" layer="1"/>
+<wire x1="18.7548" y1="14.9252" x2="19.25" y2="14.85" width="0.1524" layer="1"/>
+<wire x1="18.5596" y1="18.9976" x2="17.9" y2="19.05" width="0.1524" layer="1"/>
 </signal>
 <signal name="N$3">
 <contactref element="P4" pad="VCC"/>
 <contactref element="P1" pad="P$1"/>
-<wire x1="32.6" y1="18.2" x2="31.5" y2="18.2" width="0.8128" layer="1"/>
-<wire x1="31.5" y1="18.2" x2="29.5" y2="20.2" width="0.8128" layer="1"/>
+<wire x1="30" y1="18.2" x2="29.9" y2="18.2" width="0.8128" layer="1"/>
+<wire x1="29.9" y1="18.2" x2="27.1" y2="20.1" width="0.8128" layer="1"/>
 </signal>
 <signal name="N$15">
 <contactref element="M1" pad="D"/>
-<wire x1="24.8" y1="24.2" x2="24.3578" y2="24.2578" width="0.8128" layer="1"/>
-<wire x1="24.3578" y1="24.2578" x2="23.7" y2="23.6" width="0.8128" layer="1"/>
-<wire x1="24.384" y1="24.2316" x2="24.3578" y2="24.2578" width="0.1524" layer="1"/>
-<wire x1="24.3" y1="24.1" x2="24.384" y2="24.2316" width="0.1524" layer="1"/>
+<wire x1="23.1" y1="24.1" x2="23.5678" y2="24.2578" width="0.8128" layer="1"/>
+<wire x1="23.5678" y1="24.2578" x2="23.7" y2="23.6" width="0.8128" layer="1"/>
+<wire x1="23.634" y1="24.2016" x2="23.5678" y2="24.2578" width="0.1524" layer="1"/>
+<wire x1="22.2" y1="23.9" x2="23.634" y2="24.2016" width="0.1524" layer="1"/>
 <contactref element="P1" pad="P$2"/>
-<wire x1="29.5" y1="23.2" x2="25.2" y2="23.2" width="0.8128" layer="1"/>
-<wire x1="25.2" y1="23.2" x2="24.3" y2="24.1" width="0.8128" layer="1"/>
+<wire x1="27.1" y1="23.1" x2="25.2" y2="23.2" width="0.8128" layer="1"/>
+<wire x1="25.2" y1="23.2" x2="22.2" y2="23.9" width="0.8128" layer="1"/>
 </signal>
 </signals>
