File: base/shinobi_BLE_analog.brd (EAGLE design)
At the start: 40.5 x 35 mm, 22 parts

Commit message: Update.
Parts:
- moved C7 11.6 mm to (12.9, 19.1)
Routing:
- net P0.03: track 24.8 -> 37.0 mm
- net GND: track 177.8 -> 186.1 mm, vias 15 -> 10
- net SWDIO: track 25.3 -> 30.7 mm
- net +3V3: track 93.3 -> 88.8 mm, vias 1 -> 0
- net P0.29: track 22.5 -> 18.5 mm
- net P0.04: track 38.7 -> 35.4 mm
- net P0.16: track 14.0 -> 14.6 mm, vias 2 -> 0
- net P0.02: track 26.4 -> 25.9 mm
Other:
- board text added: "#4"
- board text added: "Rev 1.0.1"
- board text removed: "#1"
- board text removed: "Rev 1.0.0BETA"
