File: base/shinobi_BLE_connector.sch (EAGLE design)
At the start: 17 parts

Commit message: Add shinobi connector.
Parts:
- removed SV1: (no value), con-lstb:MA08-1
- added C6: 0.1uF, FaBo-Capacitor:CAPACITOR-0603
- added P1: MF-NSML600-2, FaBo-Supply:POLYSWITCH1206
- added X1: FH12-08S-1SH, con-hirose:FH12-08S-1SH
Connections:
- removed net 3V3: C3.2, S1.OUT
- new net N$5: C3.2, P1.1, S1.OUT
- net +3V3: now also C6.2, P1.2, X1-2.1; no longer SV1.2
- net GND: now also C6.1, X1-1.1; no longer SV1.1
- net P0.02: now also X1-3.1; no longer SV1.3
- net P0.03: now also X1-4.1; no longer SV1.4
- net P0.04: now also X1-5.1; no longer SV1.5
- net P0.05: now also X1-6.1; no longer SV1.6
- net P0.28: now also X1-7.1; no longer SV1.7
- net P0.29: now also X1-8.1; no longer SV1.8

Commit message: Update.
Parts:
- removed R1: (no value), FaBo-Resistors:RESISTOR-0603
- CY1: value (none) -> 32KHz
- L1: value 10nh -> 10uh
- R2: value (none) -> 220
Connections:
- net GND: no longer R1.2
- net SWCLK: no longer R1.1
Other:
- note added: "Connector"
- note added: "USB"
- note removed: "Analog"
- moved on the sheet: C2, C4, C5, C6, CY1, L1, L2, X1-1, X1-2, X1-3, X1-4, X1-5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
