File: motor/shinobi_pwm.brd (EAGLE design)
At the start: 40.5 x 35 mm, 24 parts

Commit message: Update.
Parts:
- removed ANALOG: (no value), FaBo-Template:FABO_BRICK_3PIN_S03B-PASK-2_LONG
- removed C1, C3: 130pf, FaBo-Capacitor:0603
- removed C2: 1uf, FaBo-Capacitor:0603
- removed C4, C5: 12pf, FaBo-Capacitor:0603
- removed C7: 10uf, FaBo-Capacitor:0603
- removed CY1: (no value), FaBo-Crystal:ABRACON-ABS07-32.768KHZ
- removed I2C: (no value), FaBo-Template:FABO_BRICK_I2C_S04B-PASK-2_LONG
- removed L1: 10uH, FaBo-Inductor:0603
- removed L2: 15uH, FaBo-Inductor:1812
- removed LED1: (no value), FaBo-LED:0603
- removed R4: 4.7K, FaBo-Resistors:0603
- removed SERIAL: (no value), FaBo-Template:FABO_BRICK_SERIAL_S04B-PASK-2_LONG
- removed U$3: (no value), FaBo-Logo:LOGO_FABO_S
- removed U$4: PIN-HEADER-SMT(1.27MM)2X5, gclue:PIN-HEADER-SMT(1.27MM)2X5
- removed U$5: SWICTH-4P(KMR2), gclue-test:SWITCH-4P(KMR2)
- removed UF1: (no value), FaBo-Connetor:HIROSE-UF.L
- added C10, C9: 0.1uF, FaBo-Capacitor:0603
- added C6: 100uf, resistor:153CLV-0405
- added J1: (no value), FaBo-Template:FABO_BRICK_I2C_S04B-PASK-2_LONG
- added PWM0, PWM1, PWM2: (no value), FaBo-Template:FABO_BRICK_3PIN_HEADER
- added R13, R22: 10K, FaBo-Resistors:0402
- added R16, R17, R18, R19, R20, R21: 10K, FaBo-Resistors:0603
- added U$9: PCA9685, FaBo-Motor:PCA9685
- R1, R2: value (none) -> 220
- R3: value 4.7K -> 220
- U$2: value RAYTAC-MDBT42 -> (none); device FaBo-BT:RAYTAC-MDBT42 -> FaBo-Logo:LOGO_FABO_S
- moved R1 20.4 mm to (14.4, 31.6)
- moved R3 16.3 mm to (14.3, 26.6), turned to 0 degrees
- moved U$2 16.0 mm to (34.4, 20.1)
- moved R2 4.53 mm to (14.4, 29.1)
Connections:
- removed net +3V3: ANALOG.VCC, BAT.VCC, C7.2, I2C.VCC, R3.2, R4.2, SERIAL.VCC, U$2.11, U$4.1
- removed net DCC: L1.2, U$2.10
- removed net DEC4: C2.2, L2.P$1, U$2.9
- removed net N$1: LED1.ANODE, R2.1
- removed net N$2: L1.1, L2.P$2
- removed net P0.02: U$2.15
- removed net P0.03: ANALOG.I/O, U$2.16
- removed net P0.04: U$2.17
- removed net P0.05: U$2.18
- removed net P0.06: SERIAL.TX, U$2.19
- removed net P0.07: U$2.20
- removed net P0.08: SERIAL.RX, U$2.21
- removed net P0.09: C1.2, U$2.22, UF1.GND@1, UF1.GND@2
- removed net P0.10: C3.2, U$2.23, UF1.SIG
- removed net P0.11: U$2.25
- removed net P0.12: U$2.26
- removed net P0.13: U$2.27
- removed net P0.14: U$2.28
- removed net P0.15: U$2.29
- removed net P0.16: U$2.30, U$5.2
- removed net P0.17: U$2.31
- removed net P0.18: R2.2, U$2.32
- removed net P0.19: U$2.33
- removed net P0.20: U$2.34
- removed net P0.22: U$2.38
- removed net P0.23: U$2.41
- removed net P0.24: U$2.40
- removed net P0.25: U$2.2
- removed net P0.26: I2C.SDA, R4.1, U$2.3
- removed net P0.27: I2C.SCL, R3.1, U$2.4
- removed net P0.28: U$2.5
- removed net P0.29: U$2.6
- removed net P0.30: U$2.7
- removed net P0.31: U$2.8
- removed net RESET: U$2.35
- removed net RESET1: U$4.10
- removed net SWCLK: R1.1, U$2.36, U$4.4
- removed net SWDIO: U$2.37, U$4.2
- new net LED0: R1.1, U$9.6
- new net LED1: R2.1, U$9.7
- new net LED2: R3.1, U$9.8
- new net N$10: R18.2, U$9.2
- new net N$11: R19.2, U$9.3
- new net N$12: R20.2, U$9.4
- new net N$13: R21.2, U$9.5
- new net N$14: R22.P$2, U$9.24
- new net N$9: R17.2, U$9.1
- new net PWM0: PWM0.I/O, R1.2
- new net PWM1: PWM1.I/O, R2.2
- new net PWM2: PWM2.I/O, R3.2
- new net SCL: J1.SCL, U$9.26
- new net SDA: J1.SDA, U$9.27
- new net SYS_VCC: C9.2, J1.VCC, U$9.28
- new net VCC: BAT.VCC, C10.2, C6.+, PWM0.VCC, PWM1.VCC, PWM2.VCC
- net GND: now also C10.1, C6.-, C9.1, J1.GND, PWM0.GND, PWM1.GND, PWM2.GND, R13.P$1, R16.1, R17.1, R18.1, R19.1, R20.1, R21.1, R22.P$1, U$9.14; no longer ANALOG.GND, C1.1, C2.1, C3.1, C4.1, C5.1, C7.1, I2C.GND, LED1.CATHODE, R1.2, SERIAL.GND, U$2.1, U$2.12, U$2.24, U$2.39, U$4.3, U$4.5, U$4.9, U$5.3
- net N$7: now also R16.2, U$9.23; no longer C5.2, CY1.P$2, U$2.13
- net N$8: now also R13.P$2, U$9.25; no longer C4.2, CY1.P$1, U$2.14
Routing:
- net GND: track 172.3 -> 0.00 mm, vias 15 -> 3
- net +3V3: track 98.7 -> 0.00 mm, vias 2 -> 0
- net P0.10: track 68.5 -> 0.00 mm
- net P0.27: track 39.7 -> 0.00 mm, vias 1 -> 0
- net VCC: track 0.00 -> 33.2 mm
- net P0.09: track 32.4 -> 0.00 mm
- net P0.26: track 31.5 -> 0.00 mm, vias 3 -> 0
- net SWCLK: track 28.7 -> 0.00 mm, vias 3 -> 0
- net SYS_VCC: track 0.00 -> 23.5 mm
- net N$10: track 0.00 -> 23.0 mm
- net P0.06: track 22.4 -> 0.00 mm
- net P0.03: track 20.9 -> 0.00 mm
- net SWDIO: track 18.0 -> 0.00 mm
- net N$13: track 0.00 -> 17.5 mm, vias 0 -> 2
- net N$9: track 0.00 -> 17.3 mm
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Other:
- board text added: "#6"
- board text added: "GND"
- board text added: "PWM"
- board text added: "VCC"
- board text removed: "#1"
- board text removed: "ANALOG:3"
- board text removed: "NFC:9 NFC:10"
- board text removed: "NRF"
- board text removed: "RX:8 TX:6"
- board text removed: "SCL:27 SDA:26"
